File: VikFader4530x4/VikFader4530x4.kicad_sch (KiCad schematic)
At the start: 22 parts, among them J1 vik-module-connector, J3 Conn_01x04_Pin, U1 ADS1015IDGS

Commit message: Added JLCPCB Gerber/BOM/POS files
Parts:
- U1: value ADS1015IDGS -> ADS1115IDGS
Changed lines of the file:
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@@
 			)
 		)
-		(property "Value" "ADS1015IDGS"
+		(property "Value" "ADS1115IDGS"
 			(at 47.8633 24.13 0)
 			(effects

Commit message: All three models refactored to MOSFET setup
Parts:
- removed J3: Conn_01x04_Pin, Connector_PinHeader_2.00mm:PinHeader_1x04_P2.00mm_Vertical, symbol Connector:Conn_01x04_Pin
- added J2: Conn_01x06_Pin, Connector_PinHeader_2.54mm:PinHeader_1x06_P2.54mm_Vertical, symbol Connector:Conn_01x06_Pin
- added JP1: 0x48, Jumper:SolderJumper-2_P1.3mm_Bridged_RoundedPad1.0x1.5mm, symbol Jumper:Jumper_2_Bridged
- added JP2: 0x49, Jumper:SolderJumper-2_P1.3mm_Open_RoundedPad1.0x1.5mm, symbol Jumper:Jumper_2_Open
- added JP3: 0x4A, Jumper:SolderJumper-2_P1.3mm_Open_RoundedPad1.0x1.5mm, symbol Jumper:Jumper_2_Open
- added JP4: 0x4B, Jumper:SolderJumper-2_P1.3mm_Open_RoundedPad1.0x1.5mm, symbol Jumper:Jumper_2_Open
- added Q1: DMG2305UX, Package_TO_SOT_SMD:SOT-23, symbol Transistor_FET:DMG2301L
- added R11: 1kΩ, Resistor_SMD:R_0603_1608Metric, symbol Device:R
- added R12: 100kΩ, Resistor_SMD:R_0603_1608Metric, symbol Device:R
- added R13: 10kΩ, Resistor_SMD:R_0805_2012Metric, symbol Device:R
- R2, R3: footprint Capacitor_SMD:C_0603_1608Metric -> Resistor_SMD:R_0805_2012Metric
Connections:
- net +3V3: now also J2.1 (Pin_1), JP2.2 (B), Q1.2 (S), R12.2, R13.1; no longer R1.1, R10.1, R5.1, R8.1
- net GND: now also J2.2 (Pin_2), JP1.1 (A); no longer U1.1 (ADDR)
- net GP1: now also U1.2 (ALERT/RDY), J2.5 (Pin_5), R13.2
- net GP2: now also J2.6 (Pin_6), R11.2
- net SCL: now also J2.4 (Pin_4), JP3.2 (B)
- net SDA: now also J2.3 (Pin_3), JP4.2 (B)
- new net: JP1.2 (B), JP2.1 (A), JP3.1 (A), JP4.1 (A), U1.1 (ADDR)
- new net: Q1.1 (G), R11.1, R12.1
- new net FET-OUT: Q1.3 (D), R1.1, R10.1, R5.1, R8.1
- no-connect marks 1 -> 0
Other:
- moved on the sheet: C2, J1, R2, R3
